Commit message: add rviz2 launch

File: description/urdf/camera.xacro (robot description, xacro)
@@ -38,5 +38,5 @@
         <sensor name="camera" type="camera">
             <pose> 0 0 0 0 0 0 </pose>
-            <visualize>true</visualize>
+            <visualize>false</visualize>
             <update_rate>10</update_rate>
             <camera>

File: description/urdf/ros2_control.xacro (robot description, xacro)
@@ -7,4 +7,6 @@
                 <param name="left_wheel_name">fl_wheel_joint</param>
                 <param name="right_wheel_name">fr_wheel_joint</param>
+                <param name="left_wheel_name">rl_wheel_joint</param>
+                <param name="right_wheel_name">rr_wheel_joint</param>
                 <param name="loop_rate">30</param>
                 <param name="device">/dev/serial/by-path/platform-fd500000.pcie-pci-0000:01:00.0-usb-0:1.2:1.0</param>
@@ -22,4 +24,20 @@
             </joint>
             <joint name="fr_wheel_joint">
+                <command_interface name="velocity">
+                    <param name="min">-10</param>
+                    <param name="max">10</param>
+                </command_interface>
+                <state_interface name="velocity"/>
+                <state_interface name="position"/>
+            </joint>
+            <joint name="rl_wheel_joint">
+                <command_interface name="velocity">
+                    <param name="min">-10</param>
+                    <param name="max">10</param>
+                </command_interface>
+                <state_interface name="velocity"/>
+                <state_interface name="position"/>
+            </joint>
+            <joint name="rr_wheel_joint">
                 <command_interface name="velocity">
                     <param name="min">-10</param>
