Commit message: Port to Gazebo Harmonic: consolidate launch files, add gz_bridge config, remove legacy indoor/outdoor split

File: description/urdf/camera.xacro (robot description, xacro)
@@ -41,4 +41,5 @@
             <update_rate>10</update_rate>
             <camera>
+                <camera_info_topic>camera/camera_info</camera_info_topic>
                 <horizontal_fov>1.089</horizontal_fov>
                 <image>
@@ -52,7 +53,6 @@
                 </clip>
             </camera>
-            <plugin name="camera_controller" filename="libgazebo_ros_camera.so">
-                <frame_name>camera_link_optical</frame_name>
-            </plugin>
+            <topic>camera/image_raw</topic>
+            <gz_frame_id>camera_link_optical</gz_frame_id>
         </sensor>
     </gazebo>

File: description/urdf/lidar_ld19.xacro (robot description, xacro)
@@ -31,9 +31,9 @@
     <gazebo reference="lidar_link">
         <material>Gazebo/Black</material>
-        <sensor name="laser" type="ray">
+        <sensor name="laser" type="gpu_lidar">
             <pose> 0 0 0 0 0 0 </pose>
             <visualize>true</visualize>
             <update_rate>10</update_rate>
-            <ray>
+            <lidar>
                 <scan>
                     <horizontal>
@@ -47,12 +47,7 @@
                     <max>12</max>
                 </range>
-            </ray>
-            <plugin name="laser_controller" filename="libgazebo_ros_ray_sensor.so">
-                <ros>
-                    <argument>~/out:=scan</argument>
-                </ros>
-                <output_type>sensor_msgs/LaserScan</output_type>
-                <frame_name>lidar_link</frame_name>
-            </plugin>
+            </lidar>
+                <topic>scan</topic>
+                <gz_frame_id>laser_frame</gz_frame_id>
         </sensor>
     </gazebo>

File: description/urdf/my_robot.xacro (robot description, xacro)
@@ -128,11 +128,7 @@
     <gazebo reference="fr_wheel_link">
         <material>Gazebo/Black</material>
-        <mu1 value="0.001"/>
-        <mu2 value="0.001"/>
     </gazebo>
     <gazebo reference="fl_wheel_link">
         <material>Gazebo/Black</material>
-        <mu1 value="0.001"/>
-        <mu2 value="0.001"/>
     </gazebo>
     <!-- JOINT -->
@@ -165,5 +161,4 @@
         <origin xyz="0.1 -0.1025 0" rpy="0 0 0"/>
         <axis xyz="0 1 0" />
-        <mimic joint="rr_wheel_joint" multiplier="1" offset="0"/>
     </joint>
     <joint name="fl_wheel_joint" type="continuous">
@@ -172,5 +167,4 @@
         <origin xyz="0.1 0.1025 0" rpy="0 0 0"/>
         <axis xyz="0 1 0" />
-        <mimic joint="rl_wheel_joint" multiplier="1" offset="0"/>
     </joint>
 </robot>

File: description/urdf/ros2_control.xacro (robot description, xacro)
@@ -5,6 +5,8 @@
             <hardware>
                 <plugin>diffdrive_arduino/DiffDriveArduino</plugin>
-                <param name="left_wheel_name">rl_wheel_joint</param>
-                <param name="right_wheel_name">rr_wheel_joint</param>
+                <param name="fl_wheel_name">fl_wheel_joint</param>
+                <param name="fr_wheel_name">fr_wheel_joint</param>
+                <param name="rl_wheel_name">rl_wheel_joint</param>
+                <param name="rr_wheel_name">rr_wheel_joint</param>
                 <param name="loop_rate">20</param>
                 <param name="device">/dev/serial/by-path/platform-fd500000.pcie-pci-0000:01:00.0-usb-0:1.2:1.0</param>
@@ -13,4 +15,20 @@
                 <param name="enc_counts_per_rev">1493</param>
             </hardware>
+            <joint name="fl_wheel_joint">
+                <command_interface name="velocity">
+                    <param name="min">-10</param>
+                    <param name="max">10</param>
+                </command_interface>
+                <state_interface name="velocity"/>
+                <state_interface name="position"/>
+            </joint>
+            <joint name="fr_wheel_joint">
+                <command_interface name="velocity">
+                    <param name="min">-10</param>
+                    <param name="max">10</param>
+                </command_interface>
+                <state_interface name="velocity"/>
+                <state_interface name="position"/>
+            </joint>
             <joint name="rl_wheel_joint">
                 <command_interface name="velocity">
@@ -34,6 +52,22 @@
         <ros2_control name="GazeboSystem" type="system">
             <hardware>
-                <plugin>gazebo_ros2_control/GazeboSystem</plugin>
+                <plugin>gz_ros2_control/GazeboSimSystem</plugin>
             </hardware>
+            <joint name="fl_wheel_joint">
+                <command_interface name="velocity">
+                    <param name="min">-10</param>
+                    <param name="max">10</param>
+                </command_interface>
+                <state_interface name="velocity"/>
+                <state_interface name="position"/>
+            </joint>
+            <joint name="fr_wheel_joint">
+                <command_interface name="velocity">
+                    <param name="min">-10</param>
+                    <param name="max">10</param>
+                </command_interface>
+                <state_interface name="velocity"/>
+                <state_interface name="position"/>
+            </joint>
             <joint name="rl_wheel_joint">
                 <command_interface name="velocity">
@@ -55,5 +89,5 @@
     </xacro:if>
     <gazebo>
-        <plugin name="gazebo_ros2_control" filename="libgazebo_ros2_control.so">
+        <plugin name="gz_ros2_control::GazeboSimROS2ControlPlugin" filename="libgz_ros2_control-system.so">
             <parameters>$(find tarobot_one)/config/4wheel_controllers.yaml</parameters>
             <parameters>$(find tarobot_one)/config/gaz_ros2_ctl_use_sim.yaml</parameters>
