Commit message: Modified launch file

File: description/urdf/my_robot.xacro (robot description, xacro)
@@ -12,20 +12,52 @@
     <link name="base_link">
         <visual>
-            <origin xyz="0 0 0.028" rpy="0 0 0"/>
+            <origin xyz="0 0 0.028" rpy="0 0 0" />
             <geometry>
-                <box size="0.3 0.15 0.056"/>
+                <box size="0.3 0.15 0.056" />
             </geometry>
-            <material name="blue"/>
+            <material name="blue" />
         </visual>
+        <inertial>
+            <origin xyz="0 0 0.028" rpy="0 0 0" />
+            <mass value="1.0" />
+            <inertia ixx="${(1.0/12) * (0.056*0.056 + 0.3*0.3)}" ixy="0" ixz="0"
+                     iyy="${(1.0/12) * (0.15*0.15 + 0.3*0.3)}" iyz="0"
+                     izz="${(1.0/12) * (0.15*0.15 + 0.056*0.056)}" />
+        </inertial>
+        <collision>
+            <origin xyz="0 0 0.028" rpy="0 0 0" />
+            <geometry>
+                <box size="0.3 0.15 0.056" />
+            </geometry>
+        </collision>
     </link>
+    <gazebo reference="base_link">
+        <material>Gazebo/Blue</material>
+    </gazebo>
     <link name="mid_link">
         <visual>
+            <origin xyz="0 0 0.0025" rpy="0 0 0" />
+            <geometry>
+                <box size="0.3 0.2 0.005" />
+            </geometry>
+            <material name="blue" />
+        </visual>
+        <inertial>
+            <origin xyz="0 0 0.0025" rpy="0 0 0" />
+            <mass value="0.5" />
+            <inertia ixx="${(0.5/12) * (0.005*0.005 + 0.3*0.3)}" ixy="0" ixz="0"
+                     iyy="${(0.5/12) * (0.2*0.2 + 0.3*0.3)}" iyz="0"
+                     izz="${(0.5/12) * (0.2*0.2 + 0.005*0.005)}" />
+        </inertial>
+        <collision>
             <origin xyz="0 0 0.0025" rpy="0 0 0"/>
             <geometry>
                 <box size="0.3 0.2 0.005"/>
             </geometry>
-            <material name="blue"/>
-        </visual>
+        </collision>
     </link>
+    <gazebo reference="mid_link">
+        <material>Gazebo/Blue</material>
+    </gazebo>
     <link name="top_link">
         <visual>
@@ -36,14 +68,21 @@
             <material name="blue"/>
         </visual>
+        <inertial>
+            <origin xyz="0 0 0.05" rpy="0 0 0" />
+            <mass value="2.0" />
+            <inertia ixx="${(2.0/12) * (0.1*0.1 + 0.18*0.18)}" ixy="0" ixz="0"
+                     iyy="${(2.0/12) * (0.17*0.17 + 0.18*0.18)}" iyz="0"
+                     izz="${(2.0/12) * (0.17*0.17 + 0.1*0.1)}" />
+        </inertial>
+        <collision>
+            <origin xyz="0 0 0.05" rpy="0 0 0"/>
+            <geometry>
+                <box size="0.18 0.17 0.1"/>
+            </geometry>
+        </collision>
     </link>
-    <link name="lidar_link">
-        <visual>
-            <origin xyz="0 0 0" rpy="0 0 0"/>
-            <geometry>
-                <cylinder radius="0.02" length="0.03"/>
-            </geometry>
-            <material name="black"/>
-        </visual>
-    </link>
+    <gazebo reference="top_link">
+        <material>Gazebo/Blue</material>
+    </gazebo>
     <xacro:macro name="wheel_link" params="prefix">
         <link name="${prefix}_wheel_link">
@@ -55,4 +94,17 @@
                 <material name="black" />
             </visual>
+            <inertial>
+                <origin xyz="0 0 0" rpy="${pi / 2.0} 0 0" />
+                <mass value="0.2"/>
+                <inertia ixx="${(0.2/12) * (3*0.05*0.05 + 0.035*0.035)}" ixy="0" ixz="0"
+                         iyy="${(0.2/12) * (3*0.05*0.05 + 0.035*0.035)}" iyz="0"
+                         izz="${(0.2/2) * (0.05*0.05)}" />
+            </inertial>
+            <collision>
+                <origin xyz="0 0 0" rpy="${pi / 2.0} 0 0" />
+                <geometry>
+                    <cylinder radius="0.05" length="0.035" />
+                </geometry>
+            </collision>
         </link>
     </xacro:macro>
@@ -61,13 +113,16 @@
     <xacro:wheel_link prefix="fr" />
     <xacro:wheel_link prefix="fl" />
-    <link name="camera_link">
-        <visual>
-            <origin xyz="0 0 0.0125" rpy="0 0 0"/>
-            <geometry>
-                <box size="0.015 0.07 0.025"/>
-            </geometry>
-            <material name="black"/>
-        </visual>
-    </link>
+    <gazebo reference="rr_wheel_link">
+        <material>Gazebo/Black</material>
+    </gazebo>
+    <gazebo reference="rl_wheel_link">
+        <material>Gazebo/Black</material>
+    </gazebo>
+    <gazebo reference="fr_wheel_link">
+        <material>Gazebo/Black</material>
+    </gazebo>
+    <gazebo reference="fl_wheel_link">
+        <material>Gazebo/Black</material>
+    </gazebo>
     <!-- JOINT -->
     <joint name="base_mid" type="fixed">
@@ -80,10 +135,4 @@
         <child link="top_link"/>
         <origin xyz="-0.025 0 0.005" rpy="0 0 0"/>
-    </joint>
-    <joint name="top_lidar" type="continuous">
-        <parent link="top_link"/>
-        <child link="lidar_link"/>
-        <origin xyz="0.025 0 0.115" rpy="0 0 0"/>
-        <axis xyz="0 0 -1" />
     </joint>
     <joint name="rr_wheel" type="continuous">
@@ -111,8 +160,3 @@
         <axis xyz="0 1 0" />
     </joint>
-    <joint name="mid_camera" type="fixed">
-        <parent link="mid_link"/>
-        <child link="camera_link"/>
-        <origin xyz="0.1425 0 0.005" rpy="0 0 0"/>
-    </joint>
 </robot>

File: description/urdf/robot.urdf.xacro (robot description, xacro)
@@ -1,5 +1,5 @@
 <?xml version="1.0"?>
 <robot xmlns:xacro="http://www.ros.org/wiki/xacro"  name="robot">
-    <xacro:include filename="$(find tarobot_one)/description/urdf/my_robot1.xacro" />
+    <xacro:include filename="$(find tarobot_one)/description/urdf/my_robot.xacro" />
     <xacro:include filename="$(find tarobot_one)/description/urdf/properties.xacro" />
     <xacro:include filename="$(find tarobot_one)/description/urdf/camera.xacro" />

Commit message: change description & control

File: description/urdf/my_robot.xacro (robot description, xacro)
@@ -1,4 +1,11 @@
 <?xml version="1.0"?>
 <robot xmlns:xacro="http://www.ros.org/wiki/xacro">
+    <!-- MATERIAL -->
+    <material name="blue">
+        <color rgba="0.200 0.200 1.000 1.000" />
+    </material>
+    <material name="black">
+        <color rgba="0.000 0.000 0.000 1.000" />
+    </material>
     <!-- BASE -->
     <link name="base_footprint">

File: description/urdf/robot.urdf.xacro (robot description, xacro)
@@ -1,8 +1,14 @@
 <?xml version="1.0"?>
 <robot xmlns:xacro="http://www.ros.org/wiki/xacro"  name="robot">
+    <xacro:arg name="use_ros2_control" default="false"/>
+    <xacro:arg name="sim_mode" default="true"/>
     <xacro:include filename="$(find tarobot_one)/description/urdf/my_robot.xacro" />
-    <xacro:include filename="$(find tarobot_one)/description/urdf/properties.xacro" />
     <xacro:include filename="$(find tarobot_one)/description/urdf/camera.xacro" />
     <xacro:include filename="$(find tarobot_one)/description/urdf/lidar_ld19.xacro" />
-    <xacro:include filename="$(find tarobot_one)/description/urdf/4wheel_diff.xacro" />
+    <xacro:if value="$(arg use_ros2_control)">
+        <xacro:include filename="ros2_control.xacro" />
+    </xacro:if>
+    <xacro:unless value="$(arg use_ros2_control)">
+        <xacro:include filename="4wheel_diff.xacro" />
+    </xacro:unless>
 </robot>

Commit message: control edit

File: description/urdf/my_robot.xacro (robot description, xacro)
@@ -143,5 +143,5 @@
         <origin xyz="-0.025 0 0.005" rpy="0 0 0"/>
     </joint>
-    <joint name="rr_wheel" type="continuous">
+    <joint name="rr_wheel" type="fixed">
         <parent link="base_link"/>
         <child link="rr_wheel_link"/>
@@ -149,5 +149,5 @@
         <axis xyz="0 1 0" />
     </joint>
-    <joint name="rl_wheel" type="continuous">
+    <joint name="rl_wheel" type="fixed">
         <parent link="base_link"/>
         <child link="rl_wheel_link"/>

File: description/urdf/ros2_control.xacro (robot description, xacro)
@@ -5,9 +5,6 @@
             <hardware>
                 <plugin>diffdrive_arduino/DiffDriveArduino</plugin>
-                <param name="num_wheel_pairs">2</param>
                 <param name="left_wheel_name">fl_wheel_joint</param>
                 <param name="right_wheel_name">fr_wheel_joint</param>
-                <param name="left_wheel_name">rl_wheel_joint</param>
-                <param name="right_wheel_name">rr_wheel_joint</param>
                 <param name="loop_rate">30</param>
                 <param name="device">/dev/serial/by-path/platform-fd500000.pcie-pci-0000:01:00.0-usb-0:1.2:1.0</param>
@@ -25,20 +22,4 @@
             </joint>
             <joint name="fr_wheel_joint">
-                <command_interface name="velocity">
-                    <param name="min">-10</param>
-                    <param name="max">10</param>
-                </command_interface>
-                <state_interface name="velocity"/>
-                <state_interface name="position"/>
-            </joint>
-            <joint name="rl_wheel_joint">
-                <command_interface name="velocity">
-                    <param name="min">-10</param>
-                    <param name="max">10</param>
-                </command_interface>
-                <state_interface name="velocity"/>
-                <state_interface name="position"/>
-            </joint>
-            <joint name="rr_wheel_joint">
                 <command_interface name="velocity">
                     <param name="min">-10</param>

Commit message: control edit

File: description/urdf/my_robot.xacro (robot description, xacro)
@@ -143,5 +143,5 @@
         <origin xyz="-0.025 0 0.005" rpy="0 0 0"/>
     </joint>
-    <joint name="rr_wheel" type="fixed">
+    <joint name="rr_wheel" type="continuous">
         <parent link="base_link"/>
         <child link="rr_wheel_link"/>
@@ -149,5 +149,5 @@
         <axis xyz="0 1 0" />
     </joint>
-    <joint name="rl_wheel" type="fixed">
+    <joint name="rl_wheel" type="continuous">
         <parent link="base_link"/>
         <child link="rl_wheel_link"/>

File: description/urdf/ros2_control.xacro (robot description, xacro)
@@ -5,6 +5,6 @@
             <hardware>
                 <plugin>diffdrive_arduino/DiffDriveArduino</plugin>
-                <param name="left_wheel_name">fl_wheel_joint</param>
-                <param name="right_wheel_name">fr_wheel_joint</param>
+                <param name="left_wheel_name">rl_wheel_joint</param>
+                <param name="right_wheel_name">rr_wheel_joint</param>
                 <param name="loop_rate">30</param>
                 <param name="device">/dev/serial/by-path/platform-fd500000.pcie-pci-0000:01:00.0-usb-0:1.2:1.0</param>
@@ -13,5 +13,5 @@
                 <param name="enc_counts_per_rev">3436</param>
             </hardware>
-            <joint name="fl_wheel_joint">
+            <joint name="rl_wheel_joint">
                 <command_interface name="velocity">
                     <param name="min">-10</param>
@@ -21,5 +21,5 @@
                 <state_interface name="position"/>
             </joint>
-            <joint name="fr_wheel_joint">
+            <joint name="rr_wheel_joint">
                 <command_interface name="velocity">
                     <param name="min">-10</param>
