Commit message: control edit

File: description/urdf/4wheel_diff.xacro (robot description, xacro)
@@ -1,10 +1,26 @@
 <robot xmlns:xacro="http://ros.org/wiki/xacro">
     <gazebo>
-        <plugin name="differential_drive_controller" filename="libgazebo_ros_diff_drive.so">
-            <num_wheel_pairs>2</num_wheel_pairs>
-            <left_joint>fl_wheel</left_joint>
-            <right_joint>fr_wheel</right_joint>
-            <left_joint>rl_wheel</left_joint>
-            <right_joint>rr_wheel</right_joint>
+        <plugin name="diff_drive" filename="libgazebo_ros_diff_drive.so">
+            <!-- Wheel Information -->
+            <left_joint>rl_wheel_joint</left_joint>
+            <right_joint>rr_wheel_joint</right_joint>
+            <wheel_separation>0.185</wheel_separation>
+            <wheel_diameter>0.1</wheel_diameter>
+            <!-- Limits -->
+            <max_wheel_torque>200</max_wheel_torque>
+            <max_wheel_acceleration>10.0</max_wheel_acceleration>
+            <!-- Output -->
+            <odometry_frame>odom</odometry_frame>
+            <robot_base_frame>base_footprint</robot_base_frame>
+            <publish_odom>true</publish_odom>
+            <publish_odom_tf>true</publish_odom_tf>
+            <publish_wheel_tf>true</publish_wheel_tf>
+        </plugin>
+        <!-- plugin name="differential_drive_controller" filename="libgazebo_ros_diff_drive.so">
+            <um_wheel_pairs>2</num_wheel_pairs>
+            <left_joint>fl_wheel_joint</left_joint>
+            <right_joint>fr_wheel_joint</right_joint>
+            <left_joint>rl_wheel_joint</left_joint>
+            <right_joint>rr_wheel_joint</right_joint>
             <wheel_separation>0.185</wheel_separation>
             <wheel_separation>0.185</wheel_separation>
@@ -19,5 +35,5 @@
             <odometry_frame>odom</odometry_frame>
             <robot_base_frame>base_footprint</robot_base_frame>
-        </plugin>
+        </plugin -->
     </gazebo>
 </robot>

File: description/urdf/my_robot.xacro (robot description, xacro)
@@ -128,7 +128,11 @@
     <gazebo reference="fr_wheel_link">
         <material>Gazebo/Black</material>
+        <mu1 value="0.001"/>
+        <mu2 value="0.001"/>
     </gazebo>
     <gazebo reference="fl_wheel_link">
         <material>Gazebo/Black</material>
+        <mu1 value="0.001"/>
+        <mu2 value="0.001"/>
     </gazebo>
     <!-- JOINT -->
@@ -143,5 +147,5 @@
         <origin xyz="-0.025 0 0.005" rpy="0 0 0"/>
     </joint>
-    <joint name="rr_wheel" type="continuous">
+    <joint name="rr_wheel_joint" type="continuous">
         <parent link="base_link"/>
         <child link="rr_wheel_link"/>
@@ -149,5 +153,5 @@
         <axis xyz="0 1 0" />
     </joint>
-    <joint name="rl_wheel" type="continuous">
+    <joint name="rl_wheel_joint" type="continuous">
         <parent link="base_link"/>
         <child link="rl_wheel_link"/>
@@ -155,5 +159,5 @@
         <axis xyz="0 1 0" />
     </joint>
-    <joint name="fr_wheel" type="continuous">
+    <joint name="fr_wheel_joint" type="fixed">
         <parent link="base_link"/>
         <child link="fr_wheel_link"/>
@@ -161,5 +165,5 @@
         <axis xyz="0 1 0" />
     </joint>
-    <joint name="fl_wheel" type="continuous">
+    <joint name="fl_wheel_joint" type="fixed">
         <parent link="base_link"/>
         <child link="fl_wheel_link"/>

File: description/urdf/robot.urdf.xacro (robot description, xacro)
@@ -1,6 +1,6 @@
 <?xml version="1.0"?>
 <robot xmlns:xacro="http://www.ros.org/wiki/xacro"  name="robot">
-    <xacro:arg name="use_ros2_control" default="false"/>
-    <xacro:arg name="sim_mode" default="true"/>
+    <xacro:arg name="use_ros2_control" default="true"/>
+    <xacro:arg name="sim_mode" default="false"/>
     <xacro:include filename="$(find tarobot_one)/description/urdf/my_robot.xacro" />
     <xacro:include filename="$(find tarobot_one)/description/urdf/camera.xacro" />

File: description/urdf/ros2_control.xacro (robot description, xacro)
@@ -36,20 +36,4 @@
                 <plugin>gazebo_ros2_control/GazeboSystem</plugin>
             </hardware>
-            <joint name="fl_wheel_joint">
-                <command_interface name="velocity">
-                    <param name="min">-10</param>
-                    <param name="max">10</param>
-                </command_interface>
-                <state_interface name="velocity"/>
-                <state_interface name="position"/>
-            </joint>
-            <joint name="fr_wheel_joint">
-                <command_interface name="velocity">
-                    <param name="min">-10</param>
-                    <param name="max">10</param>
-                </command_interface>
-                <state_interface name="velocity"/>
-                <state_interface name="position"/>
-            </joint>
             <joint name="rl_wheel_joint">
                 <command_interface name="velocity">
@@ -71,23 +55,4 @@
     </xacro:if>
     <gazebo>
-        <!-- plugin name="differential_drive_controller" filename="libgazebo_ros_diff_drive.so">
-            <um_wheel_pairs>2</num_wheel_pairs>
-            <left_joint>fl_wheel</left_joint>
-            <right_joint>fr_wheel</right_joint>
-            <left_joint>rl_wheel</left_joint>
-            <right_joint>rr_wheel</right_joint>
-            <wheel_separation>0.185</wheel_separation>
-            <wheel_separation>0.185</wheel_separation>
-            <wheel_diameter>0.1</wheel_diameter>
-            <wheel_diameter>0.1</wheel_diameter>
-            <updateRate>100</updateRate>
-            <max_wheel_acceleration>1.0</max_wheel_acceleration>
-            <publish_odom>true</publish_odom>
-            <publish_odom_tf>true</publish_odom_tf>
-            <publish_wheel_tf>true</publish_wheel_tf>
-            <odometry_topic>odom</odometry_topic>
-            <odometry_frame>odom</odometry_frame>
-            <robot_base_frame>base_footprint</robot_base_frame>
-        </plugin -->
         <plugin name="gazebo_ros2_control" filename="libgazebo_ros2_control.so">
             <parameters>$(find tarobot_one)/config/4wheel_controllers.yaml</parameters>

Commit message: fixed separate

File: description/urdf/4wheel_diff.xacro (robot description, xacro)
@@ -5,6 +5,6 @@
             <left_joint>rl_wheel_joint</left_joint>
             <right_joint>rr_wheel_joint</right_joint>
-            <wheel_separation>0.185</wheel_separation>
-            <wheel_diameter>0.1</wheel_diameter>
+            <wheel_separation>0.2</wheel_separation>
+            <wheel_diameter>0.1016</wheel_diameter>
             <!-- Limits -->
             <max_wheel_torque>200</max_wheel_torque>

File: description/urdf/my_robot.xacro (robot description, xacro)
@@ -97,5 +97,5 @@
                 <origin xyz="0 0 0" rpy="${pi / 2.0} 0 0" />
                 <geometry>
-                    <cylinder radius="0.05" length="0.035" />
+                    <cylinder radius="0.0508" length="0.035" />
                 </geometry>
                 <material name="black" />
@@ -104,12 +104,12 @@
                 <origin xyz="0 0 0" rpy="${pi / 2.0} 0 0" />
                 <mass value="0.2"/>
-                <inertia ixx="${(0.2/12) * (3*0.05*0.05 + 0.035*0.035)}" ixy="0" ixz="0"
-                         iyy="${(0.2/12) * (3*0.05*0.05 + 0.035*0.035)}" iyz="0"
-                         izz="${(0.2/2) * (0.05*0.05)}" />
+                <inertia ixx="${(0.2/12) * (3*0.0508*0.0508 + 0.035*0.035)}" ixy="0" ixz="0"
+                         iyy="${(0.2/12) * (3*0.0508*0.0508 + 0.035*0.035)}" iyz="0"
+                         izz="${(0.2/2) * (0.0508*0.0508)}" />
             </inertial>
             <collision>
                 <origin xyz="0 0 0" rpy="${pi / 2.0} 0 0" />
                 <geometry>
-                    <cylinder radius="0.05" length="0.035" />
+                    <cylinder radius="0.0508" length="0.035" />
                 </geometry>
             </collision>

Commit message: fixed separate

File: description/urdf/4wheel_diff.xacro (robot description, xacro)
@@ -6,5 +6,5 @@
             <right_joint>rr_wheel_joint</right_joint>
             <wheel_separation>0.2</wheel_separation>
-            <wheel_diameter>0.1016</wheel_diameter>
+            <wheel_diameter>0.1</wheel_diameter>
             <!-- Limits -->
             <max_wheel_torque>200</max_wheel_torque>

File: description/urdf/my_robot.xacro (robot description, xacro)
@@ -97,5 +97,5 @@
                 <origin xyz="0 0 0" rpy="${pi / 2.0} 0 0" />
                 <geometry>
-                    <cylinder radius="0.0508" length="0.035" />
+                    <cylinder radius="0.05" length="0.035" />
                 </geometry>
                 <material name="black" />
@@ -104,12 +104,12 @@
                 <origin xyz="0 0 0" rpy="${pi / 2.0} 0 0" />
                 <mass value="0.2"/>
-                <inertia ixx="${(0.2/12) * (3*0.0508*0.0508 + 0.035*0.035)}" ixy="0" ixz="0"
-                         iyy="${(0.2/12) * (3*0.0508*0.0508 + 0.035*0.035)}" iyz="0"
-                         izz="${(0.2/2) * (0.0508*0.0508)}" />
+                <inertia ixx="${(0.2/12) * (3*0.05*0.05 + 0.035*0.035)}" ixy="0" ixz="0"
+                         iyy="${(0.2/12) * (3*0.05*0.05 + 0.035*0.035)}" iyz="0"
+                         izz="${(0.2/2) * (0.05*0.05)}" />
             </inertial>
             <collision>
                 <origin xyz="0 0 0" rpy="${pi / 2.0} 0 0" />
                 <geometry>
-                    <cylinder radius="0.0508" length="0.035" />
+                    <cylinder radius="0.05" length="0.035" />
                 </geometry>
             </collision>
