Commit message: update config and urdf for humble

File: description/urdf/4wheel_diff.xacro (robot description, xacro)
@@ -5,5 +5,5 @@
             <left_joint>rl_wheel_joint</left_joint>
             <right_joint>rr_wheel_joint</right_joint>
-            <wheel_separation>0.2</wheel_separation>
+            <wheel_separation>0.205</wheel_separation>
             <wheel_diameter>0.1016</wheel_diameter>
             <!-- Limits -->

File: description/urdf/my_robot.xacro (robot description, xacro)
@@ -35,5 +35,5 @@
             <origin xyz="0 0 0.028" rpy="0 0 0" />
             <geometry>
-                <box size="0.3 0.15 0.056" />
+                <box size="0.3 0.165 0.056" />
             </geometry>
         </collision>
@@ -150,5 +150,5 @@
         <parent link="base_link"/>
         <child link="rr_wheel_link"/>
-        <origin xyz="-0.1 -0.0925 0" rpy="0 0 0"/>
+        <origin xyz="-0.1 -0.1025 0" rpy="0 0 0"/>
         <axis xyz="0 1 0" />
     </joint>
@@ -156,5 +156,5 @@
         <parent link="base_link"/>
         <child link="rl_wheel_link"/>
-        <origin xyz="-0.1 0.0925 0" rpy="0 0 0"/>
+        <origin xyz="-0.1 0.1025 0" rpy="0 0 0"/>
         <axis xyz="0 1 0" />
     </joint>
@@ -162,5 +162,5 @@
         <parent link="base_link"/>
         <child link="fr_wheel_link"/>
-        <origin xyz="0.1 -0.0925 0" rpy="0 0 0"/>
+        <origin xyz="0.1 -0.1025 0" rpy="0 0 0"/>
         <axis xyz="0 1 0" />
     </joint>
@@ -168,5 +168,5 @@
         <parent link="base_link"/>
         <child link="fl_wheel_link"/>
-        <origin xyz="0.1 0.0925 0" rpy="0 0 0"/>
+        <origin xyz="0.1 0.1025 0" rpy="0 0 0"/>
         <axis xyz="0 1 0" />
     </joint>
