Commit message: Update Humble stable: 4WD controllers, real robot launch files, the latest nav2/slam params

File: description/urdf/lidar_ld19.xacro (robot description, xacro)
@@ -44,5 +44,5 @@
                 </scan>
                 <range>
-                    <min>0.3</min>
+                    <min>0.02</min>
                     <max>12</max>
                 </range>

File: description/urdf/my_robot.xacro (robot description, xacro)
@@ -21,5 +21,5 @@
             <origin xyz="0 0 0.028" rpy="0 0 0" />
             <geometry>
-                <box size="0.3 0.15 0.056" />
+                <box size="0.3 0.165 0.056" />
             </geometry>
             <material name="blue" />
@@ -29,6 +29,6 @@
             <mass value="1.0" />
             <inertia ixx="${(1.0/12) * (0.056*0.056 + 0.3*0.3)}" ixy="0" ixz="0"
-                     iyy="${(1.0/12) * (0.15*0.15 + 0.3*0.3)}" iyz="0"
-                     izz="${(1.0/12) * (0.15*0.15 + 0.056*0.056)}" />
+                     iyy="${(1.0/12) * (0.165*0.165 + 0.3*0.3)}" iyz="0"
+                     izz="${(1.0/12) * (0.165*0.165 + 0.056*0.056)}" />
         </inertial>
         <collision>
@@ -159,15 +159,18 @@
         <axis xyz="0 1 0" />
     </joint>
-    <joint name="fr_wheel_joint" type="fixed">
+    <!-- FRONT WHEEL JOINTS (passive, mimic rear wheels) -->
+    <joint name="fr_wheel_joint" type="continuous">
         <parent link="base_link"/>
         <child link="fr_wheel_link"/>
         <origin xyz="0.1 -0.1025 0" rpy="0 0 0"/>
         <axis xyz="0 1 0" />
+        <mimic joint="rr_wheel_joint" multiplier="1" offset="0"/>
     </joint>
-    <joint name="fl_wheel_joint" type="fixed">
+    <joint name="fl_wheel_joint" type="continuous">
         <parent link="base_link"/>
         <child link="fl_wheel_link"/>
         <origin xyz="0.1 0.1025 0" rpy="0 0 0"/>
         <axis xyz="0 1 0" />
+        <mimic joint="rl_wheel_joint" multiplier="1" offset="0"/>
     </joint>
 </robot>

File: description/urdf/ros2_control.xacro (robot description, xacro)
@@ -7,5 +7,5 @@
                 <param name="left_wheel_name">rl_wheel_joint</param>
                 <param name="right_wheel_name">rr_wheel_joint</param>
-                <param name="loop_rate">30</param>
+                <param name="loop_rate">20</param>
                 <param name="device">/dev/serial/by-path/platform-fd500000.pcie-pci-0000:01:00.0-usb-0:1.2:1.0</param>
                 <param name="baud_rate">57600</param>
