Commit message: update using imu_bno055, new frame, and new world

File: description/urdf/imu_bno055.xacro (robot description, xacro)
@@ -1,23 +1,92 @@
 <?xml version="1.0"?>
 <robot xmlns:xacro="http://www.ros.org/wiki/xacro">
+    <link name="imu_link">
+        <visual>
+            <geometry>
+                <box size="0.02 0.02 0.005"/>
+            </geometry>
+            <material name="black">
+                <color rgba="0 0 0 1"/>
+            </material>
+        </visual>
+        <collision>
+            <geometry>
+                <box size="0.02 0.02 0.005"/>
+            </geometry>
+        </collision>
+        <inertial>
+            <mass value="0.01"/>
+            <inertia ixx="0.0000001" ixy="0" ixz="0"
+                     iyy="0.0000001" iyz="0"
+                     izz="0.0000001"/>
+        </inertial>
+    </link>
+    <joint name="imu_joint" type="fixed">
+        <parent link="top_link"/>
+        <child link="imu_link"/>
+        <origin xyz="0.025 0 -0.025" rpy="0 0 0"/>
+    </joint>
     <gazebo reference="imu_link">
         <material>Gazebo/Black</material>
-        <gravity>true</gravity>
         <sensor name="imu_sensor" type="imu">
             <always_on>true</always_on>
             <update_rate>100</update_rate>
             <visualize>true</visualize>
-            <topic>__default_topic__</topic>
-            <plugin filename="libgazebo_ros_imu_sensor.so" name="imu_plugin">
-            <topicName>imu</topicName>
-            <bodyName>imu_link</bodyName>
-            <updateRateHZ>10.0</updateRateHZ>
-            <gaussianNoise>0.0</gaussianNoise>
-            <xyzOffset>0 0 0</xyzOffset>
-            <rpyOffset>0 0 0</rpyOffset>
-            <frameName>imu_link</frameName>
-            <initialOrientationAsReference>false</initialOrientationAsReference>
-            </plugin>
-            <pose>0 0 0 0 0 0</pose>
+            <topic>imu</topic>
+            <gz_frame_id>imu_link</gz_frame_id>
+            <imu>
+                <angular_velocity>
+                    <x>
+                        <noise type="gaussian">
+                            <mean>0.0</mean>
+                            <stddev>0.0017</stddev>
+                            <bias_mean>0.0</bias_mean>
+                            <bias_stddev>5e-5</bias_stddev>
+                        </noise>
+                    </x>
+                    <y>
+                        <noise type="gaussian">
+                            <mean>0.0</mean>
+                            <stddev>0.0017</stddev>
+                            <bias_mean>0.0</bias_mean>
+                            <bias_stddev>5e-5</bias_stddev>
+                        </noise>
+                    </y>
+                    <z>
+                        <noise type="gaussian">
+                            <mean>0.0</mean>
+                            <stddev>0.0017</stddev>
+                            <bias_mean>0.0</bias_mean>
+                            <bias_stddev>5e-5</bias_stddev>
+                        </noise>
+                    </z>
+                </angular_velocity>
+                <linear_acceleration>
+                    <x>
+                        <noise type="gaussian">
+                            <mean>0.0</mean>
+                            <stddev>0.012</stddev>
+                            <bias_mean>0.0</bias_mean>
+                            <bias_stddev>0.0005</bias_stddev>
+                        </noise>
+                    </x>
+                    <y>
+                        <noise type="gaussian">
+                            <mean>0.0</mean>
+                            <stddev>0.012</stddev>
+                            <bias_mean>0.0</bias_mean>
+                            <bias_stddev>0.0005</bias_stddev>
+                        </noise>
+                    </y>
+                    <z>
+                        <noise type="gaussian">
+                            <mean>0.0</mean>
+                            <stddev>0.012</stddev>
+                            <bias_mean>0.0</bias_mean>
+                            <bias_stddev>0.0005</bias_stddev>
+                        </noise>
+                    </z>
+                </linear_acceleration>
+            </imu>
         </sensor>
     </gazebo>

File: description/urdf/robot.urdf.xacro (robot description, xacro)
@@ -6,4 +6,5 @@
     <xacro:include filename="$(find tarobot_one)/description/urdf/camera.xacro" />
     <xacro:include filename="$(find tarobot_one)/description/urdf/lidar_ld19.xacro" />
+    <xacro:include filename="$(find tarobot_one)/description/urdf/imu_bno055.xacro" />
     <xacro:if value="$(arg use_ros2_control)">
         <xacro:include filename="ros2_control.xacro" />
